Commit message: Phase 1: redesign robot model to match real robot
- Tiered enclosure: grey file compartment + split double-doors (revolute),
  open middle (4 posts + shelf), black top deck carrying lidar + blue RFID
- Ultrasonic modelled as grey HC-SR04 twin-transducer eyes
- IMU centred on base_link; lower ground clearance; correct color palette

Co-Authored-By: Claude Opus 4.8 <noreply@anthropic.com>

File: src/my_robot_description/urdf/base/base.xacro (robot description, xacro)
@@ -1,69 +1,142 @@
 <?xml version="1.0"?>
 <!--
-  Base structure:  base_footprint → base_link → body_link
-  base_footprint  : REP-105 ground-projected origin (virtual, no geometry)
-  base_link       : wheel-axis height; holds the chassis platform visual
-  body_link       : the white enclosure box above the chassis
+  Enclosure structure (chassis v3): a multi-tier file-delivery cabinet.
+  TF / link tree
+    base_footprint
+      └─ base_link                      (chassis plate, wheel-axis height)
+           ├─ compartment_link          (grey file compartment: 5 panels, open front)
+           │    ├─ door_left_link        (revolute, front-left panel)
+           │    └─ door_right_link       (revolute, front-right panel)
+           ├─ frame_link                 (4 corner posts + mid shelf, open middle)
+           └─ deck_link                  (black top board — carries lidar + RFID)
+  All fixed joints except the two doors (revolute, actuated by the door servos
+  and the OPEN_DOOR / CLOSE_DOOR mission states). Doors closed = 0 rad.
 -->
 <robot xmlns:xacro="http://www.ros.org/wiki/xacro">
   <xacro:macro name="base" params="">
-    <!-- ── base_footprint ── -->
+    <!-- ── base_footprint (REP-105 ground projection) ── -->
     <link name="base_footprint"/>
     <joint name="base_joint" type="fixed">
       <parent link="base_footprint"/>
       <child  link="base_link"/>
-      <!-- Raise by wheel_radius so base_link sits at wheel-axis height -->
       <origin xyz="0 0 ${wheel_radius}" rpy="0 0 0"/>
     </joint>
-    <!-- ── base_link ── wheel-axis height, chassis platform -->
+    <!-- ── base_link: chassis plate at wheel-axis height ── -->
     <link name="base_link">
       <visual>
-        <!--
-          Chassis plate centred half-way between base_link and ground:
-          top at z=0 (= wheel axis), bottom at z = −chassis_thickness
-        -->
         <origin xyz="0 0 ${-chassis_thickness/2.0}" rpy="0 0 0"/>
-        <geometry>
-          <box size="${body_length} ${body_width} ${chassis_thickness}"/>
-        </geometry>
+        <geometry><box size="${body_length} ${body_width} ${chassis_thickness}"/></geometry>
         <material name="chassis_grey"/>
       </visual>
       <collision>
         <origin xyz="0 0 ${-chassis_thickness/2.0}" rpy="0 0 0"/>
-        <geometry>
-          <box size="${body_length} ${body_width} ${chassis_thickness}"/>
-        </geometry>
+        <geometry><box size="${body_length} ${body_width} ${chassis_thickness}"/></geometry>
       </collision>
-      <xacro:box_inertia m="${chassis_mass}"
-                         l="${body_length}" w="${body_width}" h="${chassis_thickness}"/>
+      <xacro:box_inertia m="${chassis_mass}" l="${body_length}" w="${body_width}" h="${chassis_thickness}"/>
     </link>
-    <!-- ── body_link ── the enclosure box -->
-    <joint name="body_joint" type="fixed">
+    <!-- ── compartment_link: grey file compartment (5 panels, front open) ── -->
+    <joint name="compartment_joint" type="fixed">
       <parent link="base_link"/>
-      <child  link="body_link"/>
-      <!--
-        body_link origin is at the CENTRE of the box.
-        Box bottom = base_link level (z=0 from base_link).
-        Box top    = z = body_height = 0.535 m from base_link  →  0.600 m from ground.
-        Centre     = z = body_height/2
-      -->
-      <origin xyz="0 0 ${body_height/2.0}" rpy="0 0 0"/>
+      <child  link="compartment_link"/>
+      <origin xyz="0 0 ${compartment_center_z}" rpy="0 0 0"/>
     </joint>
-    <link name="body_link">
+    <link name="compartment_link">
+      <!-- bottom -->
+      <visual><origin xyz="0 0 ${-compartment_height/2.0}"/>
+        <geometry><box size="${body_length} ${body_width} ${panel_thickness}"/></geometry>
+        <material name="compartment_grey"/></visual>
+      <!-- top (= compartment ceiling / lower shelf) -->
+      <visual><origin xyz="0 0 ${compartment_height/2.0}"/>
+        <geometry><box size="${body_length} ${body_width} ${panel_thickness}"/></geometry>
+        <material name="compartment_grey"/></visual>
+      <!-- back (-X) -->
+      <visual><origin xyz="${-body_length/2.0} 0 0"/>
+        <geometry><box size="${panel_thickness} ${body_width} ${compartment_height}"/></geometry>
+        <material name="compartment_grey"/></visual>
+      <!-- left side (+Y) -->
+      <visual><origin xyz="0 ${body_width/2.0} 0"/>
+        <geometry><box size="${body_length} ${panel_thickness} ${compartment_height}"/></geometry>
+        <material name="compartment_grey"/></visual>
+      <!-- right side (-Y) -->
+      <visual><origin xyz="0 ${-body_width/2.0} 0"/>
+        <geometry><box size="${body_length} ${panel_thickness} ${compartment_height}"/></geometry>
+        <material name="compartment_grey"/></visual>
+      <xacro:box_inertia m="${compartment_mass}" l="${body_length}" w="${body_width}" h="${compartment_height}"/>
+    </link>
+    <!-- ── Split double-door (front +X face) ── -->
+    <!-- Left panel: hinged at the front-left vertical edge, opens outward (+θ). -->
+    <joint name="door_left_joint" type="revolute">
+      <parent link="compartment_link"/>
+      <child  link="door_left_link"/>
+      <origin xyz="${body_length/2.0} ${body_width/2.0} 0" rpy="0 0 0"/>
+      <axis xyz="0 0 1"/>
+      <limit lower="0.0" upper="1.571" effort="2.0" velocity="2.0"/>
+    </joint>
+    <link name="door_left_link">
+      <visual>
+        <origin xyz="0 ${-door_width/2.0} 0" rpy="0 0 0"/>
+        <geometry><box size="${door_thickness} ${door_width} ${door_height}"/></geometry>
+        <material name="compartment_grey"/>
+      </visual>
+    </link>
+    <!-- Right panel: hinged at the front-right vertical edge, opens outward (-θ). -->
+    <joint name="door_right_joint" type="revolute">
+      <parent link="compartment_link"/>
+      <child  link="door_right_link"/>
+      <origin xyz="${body_length/2.0} ${-body_width/2.0} 0" rpy="0 0 0"/>
+      <axis xyz="0 0 1"/>
+      <limit lower="-1.571" upper="0.0" effort="2.0" velocity="2.0"/>
+    </joint>
+    <link name="door_right_link">
+      <visual>
+        <origin xyz="0 ${door_width/2.0} 0" rpy="0 0 0"/>
+        <geometry><box size="${door_thickness} ${door_width} ${door_height}"/></geometry>
+        <material name="compartment_grey"/>
+      </visual>
+    </link>
+    <!-- ── frame_link: open middle — 4 corner posts + mid shelf board ── -->
+    <joint name="frame_joint" type="fixed">
+      <parent link="base_link"/>
+      <child  link="frame_link"/>
+      <origin xyz="0 0 0" rpy="0 0 0"/>
+    </joint>
+    <link name="frame_link">
+      <!-- 4 corner posts (spanning compartment top → deck bottom) -->
+      <xacro:property name="px" value="${body_length/2.0 - post_size/2.0}"/>
+      <xacro:property name="py" value="${body_width/2.0 - post_size/2.0}"/>
+      <visual><origin xyz="${px} ${py} ${mid_shelf_z}"/>
+        <geometry><box size="${post_size} ${post_size} ${shelf_gap}"/></geometry>
+        <material name="enclosure_black"/></visual>
+      <visual><origin xyz="${px} ${-py} ${mid_shelf_z}"/>
+        <geometry><box size="${post_size} ${post_size} ${shelf_gap}"/></geometry>
+        <material name="enclosure_black"/></visual>
+      <visual><origin xyz="${-px} ${py} ${mid_shelf_z}"/>
+        <geometry><box size="${post_size} ${post_size} ${shelf_gap}"/></geometry>
+        <material name="enclosure_black"/></visual>
+      <visual><origin xyz="${-px} ${-py} ${mid_shelf_z}"/>
+        <geometry><box size="${post_size} ${post_size} ${shelf_gap}"/></geometry>
+        <material name="enclosure_black"/></visual>
+      <!-- mid shelf board -->
+      <visual><origin xyz="0 0 ${mid_shelf_z}"/>
+        <geometry><box size="${body_length} ${body_width} ${panel_thickness}"/></geometry>
+        <material name="compartment_grey"/></visual>
+    </link>
+    <!-- ── deck_link: black top board (carries lidar + RFID) ── -->
+    <joint name="deck_joint" type="fixed">
+      <parent link="base_link"/>
+      <child  link="deck_link"/>
+      <origin xyz="0 0 ${deck_center_z}" rpy="0 0 0"/>
+    </joint>
+    <link name="deck_link">
       <visual>
         <origin xyz="0 0 0" rpy="0 0 0"/>
-        <geometry>
-          <box size="${body_length} ${body_width} ${body_height}"/>
-        </geometry>
-        <material name="white"/>
+        <geometry><box size="${body_length} ${body_width} ${deck_thickness}"/></geometry>
+        <material name="deck_black"/>
       </visual>
       <collision>
         <origin xyz="0 0 0" rpy="0 0 0"/>
-        <geometry>
-          <box size="${body_length} ${body_width} ${body_height}"/>
-        </geometry>
+        <geometry><box size="${body_length} ${body_width} ${deck_thickness}"/></geometry>
       </collision>
-      <xacro:box_inertia m="${body_mass}"
-                         l="${body_length}" w="${body_width}" h="${body_height}"/>
+      <xacro:box_inertia m="${deck_mass}" l="${body_length}" w="${body_width}" h="${deck_thickness}"/>
     </link>
   </xacro:macro>

File: src/my_robot_description/urdf/materials.xacro (robot description, xacro)
@@ -1,22 +1,38 @@
 <?xml version="1.0"?>
-<!-- Named materials used for RViz visualisation -->
+<!-- Named materials for RViz visualisation (chassis v3 palette). -->
 <robot xmlns:xacro="http://www.ros.org/wiki/xacro">
-  <material name="white">
-    <color rgba="0.92 0.92 0.92 1.0"/>
+  <!-- Enclosure / structure = black -->
+  <material name="enclosure_black">
+    <color rgba="0.08 0.08 0.09 1.0"/>
   </material>
-  <material name="chassis_grey">
-    <color rgba="0.45 0.35 0.20 1.0"/>  <!-- plywood tan -->
+  <!-- File compartment = grey -->
+  <material name="compartment_grey">
+    <color rgba="0.55 0.55 0.57 1.0"/>
   </material>
+  <!-- Top deck surface + lidar = black -->
+  <material name="deck_black">
+    <color rgba="0.10 0.10 0.11 1.0"/>
+  </material>
+  <material name="lidar_black">
+    <color rgba="0.06 0.06 0.07 1.0"/>
+  </material>
+  <!-- RFID reader = blue -->
+  <material name="rfid_blue">
+    <color rgba="0.10 0.35 0.85 1.0"/>
+  </material>
+  <!-- Ultrasonic "eyes" = grey -->
+  <material name="ultrasonic_grey">
+    <color rgba="0.60 0.60 0.62 1.0"/>
+  </material>
+  <!-- Wheels = black, hub accent -->
   <material name="wheel_black">
     <color rgba="0.10 0.10 0.10 1.0"/>
   </material>
   <material name="wheel_hub_blue">
-    <color rgba="0.20 0.20 0.80 1.0"/>  <!-- purple-blue alloy rim -->
+    <color rgba="0.20 0.20 0.80 1.0"/>
   </material>
-  <material name="caster_grey">
-    <color rgba="0.55 0.55 0.55 1.0"/>
-  </material>
-  <material name="lidar_black">
-    <color rgba="0.10 0.10 0.10 1.0"/>
+  <!-- Chassis plate (hidden, low) -->
+  <material name="chassis_grey">
+    <color rgba="0.30 0.30 0.32 1.0"/>
   </material>
 </robot>

File: src/my_robot_description/urdf/properties.xacro (robot description, xacro)
@@ -1,68 +1,65 @@
 <?xml version="1.0"?>
 <!--
-  Robot dimensional properties — single source of truth.
-  All distances in metres, masses in kg.
-  Coordinate convention (ROS REP-103):
-    X = forward,  Y = left,  Z = up
+  Robot dimensional properties — single source of truth (chassis v3, 4WD).
+  All distances in metres, masses in kg.  ROS REP-103: X fwd, Y left, Z up.
   base_link origin is at wheel-axis height above ground.
+  The enclosure is a multi-tier file-delivery cabinet (not a solid box):
+    tier 1  file compartment (grey) with a split double-door on the front
+    tier 2  open shelf framed by 4 corner posts (+ a mid shelf board)
+    tier 3  top deck (black board) carrying the lidar + RFID reader
 -->
 <robot xmlns:xacro="http://www.ros.org/wiki/xacro">
   <!-- ── Math ── -->
   <xacro:property name="PI" value="3.14159265358979323846"/>
-  <!-- ── Body / Chassis ── -->
-  <!-- Outer envelope of the white enclosure box -->
-  <xacro:property name="body_length"  value="0.400"/>   <!-- X  40 cm -->
-  <xacro:property name="body_width"   value="0.300"/>   <!-- Y  30 cm -->
-  <!--
-    body_height chosen so that:
-      ground → base_link  = wheel_radius        = 0.065 m
-      base_link → body top = body_height        = 0.535 m
-      ground → body top                         = 0.600 m  ← "60 cm to lidar"
-  -->
-  <xacro:property name="body_height"  value="0.535"/>
-  <xacro:property name="chassis_thickness" value="0.020"/>  <!-- MDF/plywood platform -->
+  <!-- ── Footprint envelope ── -->
+  <xacro:property name="body_length"  value="0.400"/>   <!-- X 40 cm -->
+  <xacro:property name="body_width"   value="0.300"/>   <!-- Y 30 cm -->
+  <xacro:property name="panel_thickness" value="0.012"/>  <!-- plywood panels/boards -->
+  <xacro:property name="chassis_thickness" value="0.020"/>
+  <!-- ── Drive wheels (130 mm Ø, 60 mm wide) ── -->
+  <xacro:property name="wheel_radius" value="0.065"/>
+  <xacro:property name="wheel_width"  value="0.060"/>
+  <xacro:property name="wheel_y_offset" value="0.165"/> <!-- centreline → wheel centre -->
+  <!-- 4WD skid-steer half-wheelbase. PLACEHOLDER: set to real front↔rear axle / 2 -->
+  <xacro:property name="wheel_x_offset" value="0.150"/>
+  <!-- ── Ground clearance (wheels lowered) ── -->
+  <!-- Chassis/compartment underside sits this far above the ground.
+       Lower value = less clearance = body sits lower around the wheels. -->
+  <xacro:property name="ground_clearance" value="0.020"/>
+  <!-- Compartment underside relative to base_link (which is at wheel_radius). -->
+  <xacro:property name="compartment_z_bottom" value="${-(wheel_radius - ground_clearance)}"/> <!-- -0.045 -->
+  <!-- ── Tier heights (stack up from compartment underside) ── -->
+  <xacro:property name="compartment_height" value="0.300"/>
+  <xacro:property name="shelf_gap"          value="0.262"/>  <!-- open middle region -->
+  <xacro:property name="deck_thickness"     value="0.018"/>
+  <xacro:property name="post_size"          value="0.020"/>  <!-- corner post cross-section -->
+  <!-- Derived Z levels (from base_link) -->
+  <xacro:property name="compartment_top_z" value="${compartment_z_bottom + compartment_height}"/>       <!-- 0.255 -->
+  <xacro:property name="compartment_center_z" value="${compartment_z_bottom + compartment_height/2.0}"/> <!-- 0.105 -->
+  <xacro:property name="mid_shelf_z" value="${compartment_top_z + shelf_gap/2.0}"/>                      <!-- 0.386 -->
+  <xacro:property name="deck_bottom_z" value="${compartment_top_z + shelf_gap}"/>                        <!-- 0.517 -->
+  <xacro:property name="deck_center_z" value="${deck_bottom_z + deck_thickness/2.0}"/>                   <!-- 0.526 -->
+  <xacro:property name="deck_top_z" value="${deck_bottom_z + deck_thickness}"/>                          <!-- 0.535 → 0.600 from ground -->
+  <!-- ── Split double-door (front face, two panels) ── -->
+  <xacro:property name="door_height"    value="0.260"/>
+  <xacro:property name="door_width"     value="0.145"/>  <!-- each panel (Y) -->
+  <xacro:property name="door_thickness" value="0.012"/>
+  <!-- ── RFID reader (MFRC522 board) ── -->
+  <xacro:property name="rfid_l" value="0.060"/>
+  <xacro:property name="rfid_w" value="0.040"/>
+  <xacro:property name="rfid_h" value="0.008"/>
+  <!-- ── HC-SR04 ultrasonic "eyes" (twin transducers) ── -->
+  <xacro:property name="us_eye_radius" value="0.008"/>
+  <xacro:property name="us_eye_length" value="0.015"/>
+  <xacro:property name="us_eye_sep"    value="0.026"/>  <!-- centre-to-centre of the two eyes -->
+  <xacro:property name="us_height_above_ground" value="0.100"/>
+  <!-- ── LTME-02A lidar (70 mm Ø, 60 mm tall) ── -->
+  <xacro:property name="lidar_radius" value="0.035"/>
+  <xacro:property name="lidar_height" value="0.060"/>
   <!-- ── Masses ── -->
   <xacro:property name="chassis_mass" value="0.500"/>
-  <xacro:property name="body_mass"    value="3.000"/>
+  <xacro:property name="compartment_mass" value="2.000"/>
+  <xacro:property name="deck_mass"    value="0.400"/>
   <xacro:property name="wheel_mass"   value="0.200"/>
-  <xacro:property name="caster_mass"  value="0.050"/>
   <xacro:property name="lidar_mass"   value="0.200"/>
-  <!-- ── Drive Wheels (130 mm Ø, 60 mm wide) ── -->
-  <xacro:property name="wheel_radius" value="0.065"/>
-  <xacro:property name="wheel_width"  value="0.060"/>
-  <!--
-    Wheel joint Y position: place wheel centre just outside body edge.
-    body_width/2 + 15 mm clearance = 0.150 + 0.015 = 0.165 m
-  -->
-  <xacro:property name="wheel_y_offset" value="0.165"/>
-  <!--
-    4WD skid-steer: longitudinal half-wheelbase (front/rear axle from centre).
-    TODO: set to the real measured front↔rear axle spacing / 2. Placeholder
-    0.150 m puts the axles 300 mm apart (near the caster positions of the
-    previous chassis). Wheels sit at x = ±wheel_x_offset.
-  -->
-  <xacro:property name="wheel_x_offset" value="0.150"/>
-  <!-- ── Caster Wheels (50 mm Ø, 20 mm wide) ── -->
-  <xacro:property name="caster_radius" value="0.025"/>
-  <xacro:property name="caster_width"  value="0.020"/>
-  <!--
-    Caster joint Z from base_link: lower it so the caster touches ground.
-      caster centre height = caster_radius = 0.025 m from ground
-      base_link height     = wheel_radius  = 0.065 m from ground
-      delta_z = 0.025 − 0.065 = −0.040 m
-  -->
-  <xacro:property name="caster_z_offset" value="-0.040"/>
-  <!-- X positions along robot body (30 mm from front/rear edge) -->
-  <xacro:property name="caster_x_front"  value=" 0.170"/>
-  <xacro:property name="caster_x_rear"   value="-0.170"/>
-  <!-- ── RPLidar (70 mm Ø cylinder, 60 mm tall) ── -->
-  <xacro:property name="lidar_radius" value="0.035"/>
-  <xacro:property name="lidar_height" value="0.060"/>
-  <!--
-    Lidar joint is at the centre-top of the body (z = body_height from base_link).
-    The laser link origin is at the centre of the cylinder:
-      z from joint = lidar_height/2 = 0.030 m
-    So lidar centre above ground = 0.065 + 0.535 + 0.030 = 0.630 m
-  -->
-  <xacro:property name="lidar_z_from_base" value="${body_height}"/>  <!-- 0.535 m -->
 </robot>

File: src/my_robot_description/urdf/robot.urdf.xacro (robot description, xacro)
@@ -2,22 +2,21 @@
 <!--
   ┌─────────────────────────────────────────────────────────────────────────┐
-  │  my_robot — 4WD Skid-Steer Robot URDF (chassis v3)                     │
+  │  my_robot — 4WD skid-steer file-delivery robot (chassis v3)             │
   │                                                                         │
-  │  TF tree                                                                │
   │  base_footprint                                                         │
   │    └─[base_joint fixed z=0.065]─► base_link                            │
-  │         ├─[body_joint fixed]──────► body_link                           │
-  │         │    └─[laser_joint cont Z]► laser      (LiDAR frame)           │
-  │         ├─[front_left_wheel_joint  cont Y]► front_left_wheel_link       │
-  │         ├─[front_right_wheel_joint cont Y]► front_right_wheel_link      │
-  │         ├─[rear_left_wheel_joint   cont Y]► rear_left_wheel_link        │
-  │         └─[rear_right_wheel_joint  cont Y]► rear_right_wheel_link       │
+  │         ├─ compartment_link (grey file compartment, split doors)        │
+  │         │    ├─ door_left_link  (revolute)                              │
+  │         │    └─ door_right_link (revolute)                              │
+  │         ├─ frame_link (open middle: 4 posts + mid shelf)                │
+  │         ├─ deck_link (black top board)                                  │
+  │         │    ├─ laser     (fixed, LTME-02A)                             │
+  │         │    └─ rfid_link  (fixed, blue MFRC522)                        │
+  │         ├─ imu_link       (centre of base)                              │
+  │         ├─ ultrasonic_link (front "eyes")                               │
+  │         ├─ front_left_wheel_link  / front_right_wheel_link  (continuous)│
+  │         └─ rear_left_wheel_link   / rear_right_wheel_link   (continuous)│
   │                                                                         │
-  │  4WD skid-steer: 4 fixed-mount drive wheels, NO casters.                │
-  │                                                                         │
-  │  Heights from ground                                                    │
-  │    base_link              0.065 m  (wheel radius)                       │
-  │    body top / laser mount 0.600 m                                       │
-  │    laser centre           0.630 m                                       │
+  │  Ground clearance lowered (wheels closer to ground). Deck top 0.60 m.   │
   └─────────────────────────────────────────────────────────────────────────┘
 -->
@@ -30,20 +29,20 @@
   <xacro:include filename="$(find my_robot_description)/urdf/base/base.xacro"/>
   <xacro:include filename="$(find my_robot_description)/urdf/wheels/drive_wheel.xacro"/>
-  <!-- caster_wheel.xacro no longer used: chassis v3 is 4WD skid-steer -->
   <xacro:include filename="$(find my_robot_description)/urdf/sensors/lidar.xacro"/>
+  <xacro:include filename="$(find my_robot_description)/urdf/sensors/rfid.xacro"/>
   <xacro:include filename="$(find my_robot_description)/urdf/sensors/imu.xacro"/>
   <xacro:include filename="$(find my_robot_description)/urdf/sensors/ultrasonic.xacro"/>
   <!-- ── Instantiate robot ── -->
-  <!-- Base structure: footprint + chassis + enclosure box -->
+  <!-- Enclosure: base + compartment + split doors + frame + deck -->
   <xacro:base/>
-  <!-- Drive wheels: 4WD skid-steer — one at each corner (front/rear × L/R) -->
+  <!-- 4WD skid-steer drive wheels (one per corner) -->
   <xacro:drive_wheel prefix="front_left"  x_pos="${wheel_x_offset}"  y_reflect=" 1"/>
   <xacro:drive_wheel prefix="front_right" x_pos="${wheel_x_offset}"  y_reflect="-1"/>
   <xacro:drive_wheel prefix="rear_left"   x_pos="${-wheel_x_offset}" y_reflect=" 1"/>
   <xacro:drive_wheel prefix="rear_right"  x_pos="${-wheel_x_offset}" y_reflect="-1"/>
-  <!-- RPLidar on top of body, frame named "laser" (sllidar_ros2 default) -->
-  <xacro:lidar/>
-  <!-- MPU9250 on the electronics deck; HC-SR04 front-low (arduino_bridge frames) -->
-  <xacro:imu/>
-  <xacro:ultrasonic/>
+  <!-- Sensors -->
+  <xacro:lidar/>        <!-- on the deck -->
+  <xacro:rfid/>         <!-- blue, deck edge -->
+  <xacro:imu/>          <!-- centre of base -->
+  <xacro:ultrasonic/>   <!-- front "eyes" -->
 </robot>
