Commit message: Phase 1: redesign robot model to match real robot
- Tiered enclosure: grey file compartment + split double-doors (revolute),
  open middle (4 posts + shelf), black top deck carrying lidar + blue RFID
- Ultrasonic modelled as grey HC-SR04 twin-transducer eyes
- IMU centred on base_link; lower ground clearance; correct color palette

Co-Authored-By: Claude Opus 4.8 <noreply@anthropic.com>

File: src/my_robot_description/urdf/sensors/imu.xacro (robot description, xacro)
@@ -1,8 +1,7 @@
 <?xml version="1.0"?>
 <!--
-  MPU9250 IMU frame (frame_id of /imu/data_raw from arduino_bridge).
-  Mounted on the electronics deck near the chassis centre, axes per REP-103
-  (X forward, Y left, Z up). If the physical module ends up rotated on the
-  deck, correct it here with the rpy of imu_joint — never in software.
+  MPU6050 IMU (frame_id of /imu/data_raw). Mounted at the CENTRE OF THE BASE
+  (base_link), axes per REP-103 (X fwd, Y left, Z up). If the physical module
+  is rotated on the deck, correct it here with imu_joint rpy — never in code.
 -->
 <robot xmlns:xacro="http://www.ros.org/wiki/xacro">
@@ -10,15 +9,13 @@
     <link name="imu_link">
       <visual>
-        <geometry>
-          <box size="0.025 0.020 0.005"/>
-        </geometry>
-        <material name="lidar_black"/>
+        <geometry><box size="0.025 0.020 0.005"/></geometry>
+        <material name="enclosure_black"/>
       </visual>
     </link>
     <joint name="imu_joint" type="fixed">
-      <parent link="body_link"/>
+      <parent link="base_link"/>
       <child  link="imu_link"/>
-      <!-- 5 cm above the chassis platform, centred -->
-      <origin xyz="0 0 ${-body_height/2.0 + 0.05}" rpy="0 0 0"/>
+      <!-- Centre of the base, just above the chassis plate. -->
+      <origin xyz="0 0 0.008" rpy="0 0 0"/>
     </joint>
   </xacro:macro>

File: src/my_robot_description/urdf/sensors/lidar.xacro (robot description, xacro)
@@ -1,16 +1,9 @@
 <?xml version="1.0"?>
 <!--
-  RPLidar / SLAMTEC spinning lidar macro.
-  The link is named "laser" to match the default frame_id used by sllidar_ros2.
-  joint type = continuous so the spinning motion is visible in RViz when
-  joint_state_publisher_gui is running.
-  For real-hardware nav2 use:
-    • sllidar_ros2 already de-rotates the scan data internally — the "laser"
-      frame can stay at 0 rad; joint_state_publisher will publish 0 for it.
-    • Alternatively change joint type to "fixed" if you prefer no joint state
-      dependency.
-  Mounted at the centre of the body_link top surface:
-    z from base_link = body_height = 0.535 m  →  0.600 m from ground.
-  Lidar centre is then 0.600 + lidar_height/2 = 0.630 m from ground.
+  LTME-02A lidar on the top deck. Frame "laser" (driver frame_id).
+  FIXED joint: the frame does not rotate in real use (driver outputs
+  de-rotated scans) so base->laser is on /tf_static — a continuous joint
+  would ride dynamic /tf at the joint-state rate and cause the 30 Hz scans
+  to be dropped by SLAM/Nav2.
 -->
 <robot xmlns:xacro="http://www.ros.org/wiki/xacro">
@@ -18,40 +11,19 @@
     <link name="laser">
       <visual>
-        <!--
-          Visual origin at lidar_height/2 so the bottom of the cylinder
-          sits on the body top surface.
-        -->
         <origin xyz="0 0 ${lidar_height/2.0}" rpy="0 0 0"/>
-        <geometry>
-          <cylinder radius="${lidar_radius}" length="${lidar_height}"/>
-        </geometry>
+        <geometry><cylinder radius="${lidar_radius}" length="${lidar_height}"/></geometry>
         <material name="lidar_black"/>
       </visual>
       <collision>
         <origin xyz="0 0 ${lidar_height/2.0}" rpy="0 0 0"/>
-        <geometry>
-          <cylinder radius="${lidar_radius}" length="${lidar_height}"/>
-        </geometry>
+        <geometry><cylinder radius="${lidar_radius}" length="${lidar_height}"/></geometry>
       </collision>
-      <!-- Cylinder spinning around Z -->
       <xacro:cylinder_inertia_z m="${lidar_mass}" r="${lidar_radius}" h="${lidar_height}"/>
     </link>
-    <!--
-      FIXED joint: the lidar frame does not rotate in real use (the driver
-      outputs de-rotated scans), so base->laser belongs on /tf_static —
-      valid for every timestamp. A continuous joint would put base->laser
-      on dynamic /tf at the joint_state_publisher rate (10 Hz); the 30 Hz
-      LTME-02A scans then arrive stamped newer than the latest laser TF and
-      SLAM/Nav2 drop them ("transform queue full"). Fixed removes that rate
-      dependency entirely.
-    -->
+    <!-- Mounted on the deck top surface, centred (270° FOV faces forward). -->
     <joint name="laser_joint" type="fixed">
-      <parent link="body_link"/>
+      <parent link="deck_link"/>
       <child  link="laser"/>
-      <!--
-        body_link origin is at the body centre.
-        body_height/2 brings us to the top surface of the body.
-      -->
-      <origin xyz="0 0 ${body_height/2.0}" rpy="0 0 0"/>
+      <origin xyz="0 0 ${deck_thickness/2.0}" rpy="0 0 0"/>
     </joint>
   </xacro:macro>

File: src/my_robot_description/urdf/sensors/ultrasonic.xacro (robot description, xacro)
@@ -1,28 +1,30 @@
 <?xml version="1.0"?>
 <!--
-  HC-SR04 ultrasonic frame (frame_id of /ultrasonic/range from arduino_bridge).
-  Front face of the body, ~10 cm above ground, pointing forward (+X):
-  covers the low zone under the lidar's 0.63 m scan plane where chair legs,
-  door stops and stair edges hide.
+  HC-SR04 ultrasonic on the compartment front face, ~10 cm above ground,
+  pointing forward (+X). Modelled as the sensor's twin transducers — two
+  grey "eyes". Frame "ultrasonic_link" (frame_id of /ultrasonic/range) sits
+  at the pair centre with +X = measurement direction.
 -->
 <robot xmlns:xacro="http://www.ros.org/wiki/xacro">
   <xacro:macro name="ultrasonic" params="">
     <link name="ultrasonic_link">
+      <!-- left eye -->
       <visual>
-        <geometry>
-          <box size="0.010 0.045 0.020"/>
-        </geometry>
-        <material name="lidar_black"/>
+        <origin xyz="0 ${us_eye_sep/2.0} 0" rpy="0 ${PI/2.0} 0"/>
+        <geometry><cylinder radius="${us_eye_radius}" length="${us_eye_length}"/></geometry>
+        <material name="ultrasonic_grey"/>
+      </visual>
+      <!-- right eye -->
+      <visual>
+        <origin xyz="0 ${-us_eye_sep/2.0} 0" rpy="0 ${PI/2.0} 0"/>
+        <geometry><cylinder radius="${us_eye_radius}" length="${us_eye_length}"/></geometry>
+        <material name="ultrasonic_grey"/>
       </visual>
     </link>
     <joint name="ultrasonic_joint" type="fixed">
-      <parent link="body_link"/>
+      <parent link="base_link"/>
       <child  link="ultrasonic_link"/>
-      <!--
-        x: front face of the body.
-        z: body_link centre is 0.3325 m above ground; 0.035 above the
-           chassis-bottom edge puts the sensor 0.10 m above ground.
-      -->
-      <origin xyz="${body_length/2.0} 0 ${-body_height/2.0 + 0.035}" rpy="0 0 0"/>
+      <!-- x: compartment front face; z: us_height_above_ground − wheel_radius -->
+      <origin xyz="${body_length/2.0} 0 ${us_height_above_ground - wheel_radius}" rpy="0 0 0"/>
     </joint>
   </xacro:macro>
