Commit message: Phase 1 revision: black bottom box, grey split-door compartment (middle), black deck; RFID centred; HC-SR04 look; minimal TF (structural geometry merged onto base_link)
Co-Authored-By: Claude Opus 4.8 <noreply@anthropic.com>

File: src/my_robot_description/urdf/base/base.xacro (robot description, xacro)
@@ -1,15 +1,14 @@
 <?xml version="1.0"?>
 <!--
-  Enclosure structure (chassis v3): a multi-tier file-delivery cabinet.
-  TF / link tree
-    base_footprint
-      └─ base_link                      (chassis plate, wheel-axis height)
-           ├─ compartment_link          (grey file compartment: 5 panels, open front)
-           │    ├─ door_left_link        (revolute, front-left panel)
-           │    └─ door_right_link       (revolute, front-right panel)
-           ├─ frame_link                 (4 corner posts + mid shelf, open middle)
-           └─ deck_link                  (black top board — carries lidar + RFID)
-  All fixed joints except the two doors (revolute, actuated by the door servos
-  and the OPEN_DOOR / CLOSE_DOOR mission states). Doors closed = 0 rad.
+  Enclosure structure (chassis v3): a 3-tier file-delivery cabinet.
+  ALL static geometry is carried as multiple <visual> elements on base_link,
+  so it adds NO extra TF frames. Only the two doors (which move) get their own
+  links/frames.
+    tier 1  BLACK solid box     (bottom, no doors)
+    tier 2  GREY file compartment (hollow, open front) + split double-door
+    tier 3  BLACK deck board     (top surface; lidar + centred RFID sit on it)
+  TF frames from this file: base_footprint, base_link, door_left_link,
+  door_right_link.  (laser / imu_link / ultrasonic_link / wheels come from the
+  sensor & wheel macros.)
 -->
 <robot xmlns:xacro="http://www.ros.org/wiki/xacro">
@@ -22,121 +21,67 @@
       <origin xyz="0 0 ${wheel_radius}" rpy="0 0 0"/>
     </joint>
-    <!-- ── base_link: chassis plate at wheel-axis height ── -->
+    <!-- ── base_link: carries the whole static enclosure ── -->
     <link name="base_link">
-      <visual>
-        <origin xyz="0 0 ${-chassis_thickness/2.0}" rpy="0 0 0"/>
+      <!-- chassis plate -->
+      <visual><origin xyz="0 0 ${-chassis_thickness/2.0}"/>
         <geometry><box size="${body_length} ${body_width} ${chassis_thickness}"/></geometry>
-        <material name="chassis_grey"/>
-      </visual>
-      <collision>
-        <origin xyz="0 0 ${-chassis_thickness/2.0}" rpy="0 0 0"/>
-        <geometry><box size="${body_length} ${body_width} ${chassis_thickness}"/></geometry>
+        <material name="chassis_grey"/></visual>
+      <!-- tier 1: solid BLACK bottom box -->
+      <visual><origin xyz="0 0 ${bottom_black_center_z}"/>
+        <geometry><box size="${body_length} ${body_width} ${bottom_black_h}"/></geometry>
+        <material name="enclosure_black"/></visual>
+      <!-- tier 2: GREY file compartment — 5 panels, front open for the doors -->
+      <visual><origin xyz="0 0 ${compartment_center_z - compartment_h/2.0}"/>
+        <geometry><box size="${body_length} ${body_width} ${panel_thickness}"/></geometry>
+        <material name="compartment_grey"/></visual>                       <!-- floor -->
+      <visual><origin xyz="0 0 ${compartment_center_z + compartment_h/2.0}"/>
+        <geometry><box size="${body_length} ${body_width} ${panel_thickness}"/></geometry>
+        <material name="compartment_grey"/></visual>                       <!-- ceiling -->
+      <visual><origin xyz="${-body_length/2.0} 0 ${compartment_center_z}"/>
+        <geometry><box size="${panel_thickness} ${body_width} ${compartment_h}"/></geometry>
+        <material name="compartment_grey"/></visual>                       <!-- back -->
+      <visual><origin xyz="0 ${body_width/2.0} ${compartment_center_z}"/>
+        <geometry><box size="${body_length} ${panel_thickness} ${compartment_h}"/></geometry>
+        <material name="compartment_grey"/></visual>                       <!-- left -->
+      <visual><origin xyz="0 ${-body_width/2.0} ${compartment_center_z}"/>
+        <geometry><box size="${body_length} ${panel_thickness} ${compartment_h}"/></geometry>
+        <material name="compartment_grey"/></visual>                       <!-- right -->
+      <!-- tier 3: BLACK deck board (top surface) -->
+      <visual><origin xyz="0 0 ${deck_center_z}"/>
+        <geometry><box size="${body_length} ${body_width} ${deck_h}"/></geometry>
+        <material name="deck_black"/></visual>
+      <!-- RFID reader (blue), centred on the deck front-edge line -->
+      <visual><origin xyz="${rfid_x} 0 ${deck_top_z + rfid_h/2.0}"/>
+        <geometry><box size="${rfid_l} ${rfid_w} ${rfid_h}"/></geometry>
+        <material name="rfid_blue"/></visual>
+      <collision><origin xyz="0 0 ${compartment_center_z}"/>
+        <geometry><box size="${body_length} ${body_width} ${deck_top_z - struct_bottom_z}"/></geometry>
       </collision>
-      <xacro:box_inertia m="${chassis_mass}" l="${body_length}" w="${body_width}" h="${chassis_thickness}"/>
+      <xacro:box_inertia m="${body_mass}" l="${body_length}" w="${body_width}" h="${deck_top_z - struct_bottom_z}"/>
     </link>
-    <!-- ── compartment_link: grey file compartment (5 panels, front open) ── -->
-    <joint name="compartment_joint" type="fixed">
+    <!-- ── Split double-door on the GREY compartment front (+X) ── -->
+    <joint name="door_left_joint" type="revolute">
       <parent link="base_link"/>
-      <child  link="compartment_link"/>
-      <origin xyz="0 0 ${compartment_center_z}" rpy="0 0 0"/>
-    </joint>
-    <link name="compartment_link">
-      <!-- bottom -->
-      <visual><origin xyz="0 0 ${-compartment_height/2.0}"/>
-        <geometry><box size="${body_length} ${body_width} ${panel_thickness}"/></geometry>
-        <material name="compartment_grey"/></visual>
-      <!-- top (= compartment ceiling / lower shelf) -->
-      <visual><origin xyz="0 0 ${compartment_height/2.0}"/>
-        <geometry><box size="${body_length} ${body_width} ${panel_thickness}"/></geometry>
-        <material name="compartment_grey"/></visual>
-      <!-- back (-X) -->
-      <visual><origin xyz="${-body_length/2.0} 0 0"/>
-        <geometry><box size="${panel_thickness} ${body_width} ${compartment_height}"/></geometry>
-        <material name="compartment_grey"/></visual>
-      <!-- left side (+Y) -->
-      <visual><origin xyz="0 ${body_width/2.0} 0"/>
-        <geometry><box size="${body_length} ${panel_thickness} ${compartment_height}"/></geometry>
-        <material name="compartment_grey"/></visual>
-      <!-- right side (-Y) -->
-      <visual><origin xyz="0 ${-body_width/2.0} 0"/>
-        <geometry><box size="${body_length} ${panel_thickness} ${compartment_height}"/></geometry>
-        <material name="compartment_grey"/></visual>
-      <xacro:box_inertia m="${compartment_mass}" l="${body_length}" w="${body_width}" h="${compartment_height}"/>
-    </link>
-    <!-- ── Split double-door (front +X face) ── -->
-    <!-- Left panel: hinged at the front-left vertical edge, opens outward (+θ). -->
-    <joint name="door_left_joint" type="revolute">
-      <parent link="compartment_link"/>
       <child  link="door_left_link"/>
-      <origin xyz="${body_length/2.0} ${body_width/2.0} 0" rpy="0 0 0"/>
+      <origin xyz="${body_length/2.0} ${body_width/2.0} ${compartment_center_z}" rpy="0 0 0"/>
       <axis xyz="0 0 1"/>
       <limit lower="0.0" upper="1.571" effort="2.0" velocity="2.0"/>
     </joint>
     <link name="door_left_link">
-      <visual>
-        <origin xyz="0 ${-door_width/2.0} 0" rpy="0 0 0"/>
+      <visual><origin xyz="0 ${-door_width/2.0} 0"/>
         <geometry><box size="${door_thickness} ${door_width} ${door_height}"/></geometry>
-        <material name="compartment_grey"/>
-      </visual>
+        <material name="compartment_grey"/></visual>
     </link>
-    <!-- Right panel: hinged at the front-right vertical edge, opens outward (-θ). -->
     <joint name="door_right_joint" type="revolute">
-      <parent link="compartment_link"/>
+      <parent link="base_link"/>
       <child  link="door_right_link"/>
-      <origin xyz="${body_length/2.0} ${-body_width/2.0} 0" rpy="0 0 0"/>
+      <origin xyz="${body_length/2.0} ${-body_width/2.0} ${compartment_center_z}" rpy="0 0 0"/>
       <axis xyz="0 0 1"/>
       <limit lower="-1.571" upper="0.0" effort="2.0" velocity="2.0"/>
     </joint>
     <link name="door_right_link">
-      <visual>
-        <origin xyz="0 ${door_width/2.0} 0" rpy="0 0 0"/>
+      <visual><origin xyz="0 ${door_width/2.0} 0"/>
         <geometry><box size="${door_thickness} ${door_width} ${door_height}"/></geometry>
-        <material name="compartment_grey"/>
-      </visual>
-    </link>
-    <!-- ── frame_link: open middle — 4 corner posts + mid shelf board ── -->
-    <joint name="frame_joint" type="fixed">
-      <parent link="base_link"/>
-      <child  link="frame_link"/>
-      <origin xyz="0 0 0" rpy="0 0 0"/>
-    </joint>
-    <link name="frame_link">
-      <!-- 4 corner posts (spanning compartment top → deck bottom) -->
-      <xacro:property name="px" value="${body_length/2.0 - post_size/2.0}"/>
-      <xacro:property name="py" value="${body_width/2.0 - post_size/2.0}"/>
-      <visual><origin xyz="${px} ${py} ${mid_shelf_z}"/>
-        <geometry><box size="${post_size} ${post_size} ${shelf_gap}"/></geometry>
-        <material name="enclosure_black"/></visual>
-      <visual><origin xyz="${px} ${-py} ${mid_shelf_z}"/>
-        <geometry><box size="${post_size} ${post_size} ${shelf_gap}"/></geometry>
-        <material name="enclosure_black"/></visual>
-      <visual><origin xyz="${-px} ${py} ${mid_shelf_z}"/>
-        <geometry><box size="${post_size} ${post_size} ${shelf_gap}"/></geometry>
-        <material name="enclosure_black"/></visual>
-      <visual><origin xyz="${-px} ${-py} ${mid_shelf_z}"/>
-        <geometry><box size="${post_size} ${post_size} ${shelf_gap}"/></geometry>
-        <material name="enclosure_black"/></visual>
-      <!-- mid shelf board -->
-      <visual><origin xyz="0 0 ${mid_shelf_z}"/>
-        <geometry><box size="${body_length} ${body_width} ${panel_thickness}"/></geometry>
         <material name="compartment_grey"/></visual>
-    </link>
-    <!-- ── deck_link: black top board (carries lidar + RFID) ── -->
-    <joint name="deck_joint" type="fixed">
-      <parent link="base_link"/>
-      <child  link="deck_link"/>
-      <origin xyz="0 0 ${deck_center_z}" rpy="0 0 0"/>
-    </joint>
-    <link name="deck_link">
-      <visual>
-        <origin xyz="0 0 0" rpy="0 0 0"/>
-        <geometry><box size="${body_length} ${body_width} ${deck_thickness}"/></geometry>
-        <material name="deck_black"/>
-      </visual>
-      <collision>
-        <origin xyz="0 0 0" rpy="0 0 0"/>
-        <geometry><box size="${body_length} ${body_width} ${deck_thickness}"/></geometry>
-      </collision>
-      <xacro:box_inertia m="${deck_mass}" l="${body_length}" w="${body_width}" h="${deck_thickness}"/>
     </link>
   </xacro:macro>

File: src/my_robot_description/urdf/materials.xacro (robot description, xacro)
@@ -2,9 +2,9 @@
 <!-- Named materials for RViz visualisation (chassis v3 palette). -->
 <robot xmlns:xacro="http://www.ros.org/wiki/xacro">
-  <!-- Enclosure / structure = black -->
+  <!-- Enclosure / bottom box / structure = black -->
   <material name="enclosure_black">
     <color rgba="0.08 0.08 0.09 1.0"/>
   </material>
-  <!-- File compartment = grey -->
+  <!-- File compartment (middle tier) + split doors = grey -->
   <material name="compartment_grey">
     <color rgba="0.55 0.55 0.57 1.0"/>
@@ -21,7 +21,13 @@
     <color rgba="0.10 0.35 0.85 1.0"/>
   </material>
-  <!-- Ultrasonic "eyes" = grey -->
-  <material name="ultrasonic_grey">
-    <color rgba="0.60 0.60 0.62 1.0"/>
+  <!-- HC-SR04: blue PCB, black transducers, silver crystal -->
+  <material name="us_pcb_blue">
+    <color rgba="0.12 0.45 0.75 1.0"/>
+  </material>
+  <material name="us_transducer_black">
+    <color rgba="0.05 0.05 0.05 1.0"/>
+  </material>
+  <material name="crystal_silver">
+    <color rgba="0.75 0.76 0.78 1.0"/>
   </material>
   <!-- Wheels = black, hub accent -->

File: src/my_robot_description/urdf/properties.xacro (robot description, xacro)
@@ -4,8 +4,12 @@
   All distances in metres, masses in kg.  ROS REP-103: X fwd, Y left, Z up.
   base_link origin is at wheel-axis height above ground.
-  The enclosure is a multi-tier file-delivery cabinet (not a solid box):
-    tier 1  file compartment (grey) with a split double-door on the front
-    tier 2  open shelf framed by 4 corner posts (+ a mid shelf board)
-    tier 3  top deck (black board) carrying the lidar + RFID reader
+  Enclosure (bottom → top):
+    tier 1  solid BLACK box (no doors)
+    tier 2  GREY file compartment (hollow) with a split double-door on the front
+    tier 3  BLACK top deck (surface) carrying the lidar + centred RFID reader
+  Minimal TF: all static structure lives on base_link (multiple visuals) so it
+  produces NO extra TF frames. Only functional links get their own frame:
+  base_footprint, base_link, laser, imu_link, ultrasonic_link, the 4 wheels,
+  and the 2 (moving) doors.
 -->
 <robot xmlns:xacro="http://www.ros.org/wiki/xacro">
@@ -15,42 +19,42 @@
   <xacro:property name="body_length"  value="0.400"/>   <!-- X 40 cm -->
   <xacro:property name="body_width"   value="0.300"/>   <!-- Y 30 cm -->
-  <xacro:property name="panel_thickness" value="0.012"/>  <!-- plywood panels/boards -->
+  <xacro:property name="panel_thickness" value="0.012"/>
   <xacro:property name="chassis_thickness" value="0.020"/>
   <!-- ── Drive wheels (130 mm Ø, 60 mm wide) ── -->
   <xacro:property name="wheel_radius" value="0.065"/>
   <xacro:property name="wheel_width"  value="0.060"/>
-  <xacro:property name="wheel_y_offset" value="0.165"/> <!-- centreline → wheel centre -->
-  <!-- 4WD skid-steer half-wheelbase. PLACEHOLDER: set to real front↔rear axle / 2 -->
+  <xacro:property name="wheel_y_offset" value="0.165"/>
+  <!-- 4WD skid-steer half-wheelbase. PLACEHOLDER: real front↔rear axle / 2 -->
   <xacro:property name="wheel_x_offset" value="0.150"/>
   <!-- ── Ground clearance (wheels lowered) ── -->
-  <!-- Chassis/compartment underside sits this far above the ground.
-       Lower value = less clearance = body sits lower around the wheels. -->
   <xacro:property name="ground_clearance" value="0.020"/>
-  <!-- Compartment underside relative to base_link (which is at wheel_radius). -->
-  <xacro:property name="compartment_z_bottom" value="${-(wheel_radius - ground_clearance)}"/> <!-- -0.045 -->
-  <!-- ── Tier heights (stack up from compartment underside) ── -->
-  <xacro:property name="compartment_height" value="0.300"/>
-  <xacro:property name="shelf_gap"          value="0.262"/>  <!-- open middle region -->
-  <xacro:property name="deck_thickness"     value="0.018"/>
-  <xacro:property name="post_size"          value="0.020"/>  <!-- corner post cross-section -->
-  <!-- Derived Z levels (from base_link) -->
-  <xacro:property name="compartment_top_z" value="${compartment_z_bottom + compartment_height}"/>       <!-- 0.255 -->
-  <xacro:property name="compartment_center_z" value="${compartment_z_bottom + compartment_height/2.0}"/> <!-- 0.105 -->
-  <xacro:property name="mid_shelf_z" value="${compartment_top_z + shelf_gap/2.0}"/>                      <!-- 0.386 -->
-  <xacro:property name="deck_bottom_z" value="${compartment_top_z + shelf_gap}"/>                        <!-- 0.517 -->
-  <xacro:property name="deck_center_z" value="${deck_bottom_z + deck_thickness/2.0}"/>                   <!-- 0.526 -->
-  <xacro:property name="deck_top_z" value="${deck_bottom_z + deck_thickness}"/>                          <!-- 0.535 → 0.600 from ground -->
-  <!-- ── Split double-door (front face, two panels) ── -->
-  <xacro:property name="door_height"    value="0.260"/>
-  <xacro:property name="door_width"     value="0.145"/>  <!-- each panel (Y) -->
+  <xacro:property name="struct_bottom_z" value="${-(wheel_radius - ground_clearance)}"/> <!-- -0.045 -->
+  <!-- ── Tier heights (stack up from struct_bottom_z) ── -->
+  <xacro:property name="bottom_black_h" value="0.245"/>
+  <xacro:property name="compartment_h"  value="0.317"/>   <!-- grey file compartment -->
+  <xacro:property name="deck_h"         value="0.018"/>
+  <!-- Derived Z centres/levels (from base_link) -->
+  <xacro:property name="bottom_black_center_z" value="${struct_bottom_z + bottom_black_h/2.0}"/>          <!-- 0.0775 -->
+  <xacro:property name="bottom_black_top_z"    value="${struct_bottom_z + bottom_black_h}"/>              <!-- 0.200 -->
+  <xacro:property name="compartment_center_z"  value="${bottom_black_top_z + compartment_h/2.0}"/>        <!-- 0.3585 -->
+  <xacro:property name="compartment_top_z"     value="${bottom_black_top_z + compartment_h}"/>            <!-- 0.517 -->
+  <xacro:property name="deck_center_z"         value="${compartment_top_z + deck_h/2.0}"/>                <!-- 0.526 -->
+  <xacro:property name="deck_top_z"            value="${compartment_top_z + deck_h}"/>                    <!-- 0.535 → 0.600 ground -->
+  <!-- ── Split double-door (front of the GREY middle compartment) ── -->
+  <xacro:property name="door_height"    value="0.280"/>
+  <xacro:property name="door_width"     value="0.145"/>   <!-- each panel (Y) -->
   <xacro:property name="door_thickness" value="0.012"/>
-  <!-- ── RFID reader (MFRC522 board) ── -->
+  <!-- ── RFID reader (MFRC522) — centred on the deck front-edge line ── -->
   <xacro:property name="rfid_l" value="0.060"/>
   <xacro:property name="rfid_w" value="0.040"/>
   <xacro:property name="rfid_h" value="0.008"/>
-  <!-- ── HC-SR04 ultrasonic "eyes" (twin transducers) ── -->
-  <xacro:property name="us_eye_radius" value="0.008"/>
-  <xacro:property name="us_eye_length" value="0.015"/>
-  <xacro:property name="us_eye_sep"    value="0.026"/>  <!-- centre-to-centre of the two eyes -->
+  <xacro:property name="rfid_x" value="${body_length/2.0 - rfid_l/2.0 - 0.02}"/>  <!-- front-edge line -->
+  <!-- ── HC-SR04 ultrasonic (blue PCB + 2 black transducers + silver crystal) ── -->
+  <xacro:property name="us_pcb_w"    value="0.045"/>   <!-- board Y -->
+  <xacro:property name="us_pcb_h"    value="0.020"/>   <!-- board Z -->
+  <xacro:property name="us_pcb_t"    value="0.0015"/>  <!-- board X (thin) -->
+  <xacro:property name="us_tx_radius" value="0.008"/>  <!-- transducer can -->
+  <xacro:property name="us_tx_length" value="0.012"/>
+  <xacro:property name="us_tx_sep"    value="0.026"/>  <!-- centre-to-centre -->
   <xacro:property name="us_height_above_ground" value="0.100"/>
   <!-- ── LTME-02A lidar (70 mm Ø, 60 mm tall) ── -->
@@ -58,8 +62,6 @@
   <xacro:property name="lidar_height" value="0.060"/>
   <!-- ── Masses ── -->
-  <xacro:property name="chassis_mass" value="0.500"/>
-  <xacro:property name="compartment_mass" value="2.000"/>
-  <xacro:property name="deck_mass"    value="0.400"/>
-  <xacro:property name="wheel_mass"   value="0.200"/>
-  <xacro:property name="lidar_mass"   value="0.200"/>
+  <xacro:property name="body_mass"  value="3.000"/>
+  <xacro:property name="wheel_mass" value="0.200"/>
+  <xacro:property name="lidar_mass" value="0.200"/>
 </robot>

File: src/my_robot_description/urdf/robot.urdf.xacro (robot description, xacro)
@@ -4,19 +4,18 @@
   │  my_robot — 4WD skid-steer file-delivery robot (chassis v3)             │
   │                                                                         │
+  │  Minimal TF tree (only functional frames):                             │
   │  base_footprint                                                         │
-  │    └─[base_joint fixed z=0.065]─► base_link                            │
-  │         ├─ compartment_link (grey file compartment, split doors)        │
-  │         │    ├─ door_left_link  (revolute)                              │
-  │         │    └─ door_right_link (revolute)                              │
-  │         ├─ frame_link (open middle: 4 posts + mid shelf)                │
-  │         ├─ deck_link (black top board)                                  │
-  │         │    ├─ laser     (fixed, LTME-02A)                             │
-  │         │    └─ rfid_link  (fixed, blue MFRC522)                        │
-  │         ├─ imu_link       (centre of base)                              │
-  │         ├─ ultrasonic_link (front "eyes")                               │
-  │         ├─ front_left_wheel_link  / front_right_wheel_link  (continuous)│
-  │         └─ rear_left_wheel_link   / rear_right_wheel_link   (continuous)│
+  │    └─[base_joint fixed z=0.065]─► base_link  (carries ALL static        │
+  │         │                          geometry: black bottom box, grey     │
+  │         │                          file compartment, black deck, RFID)  │
+  │         ├─ laser            (fixed, LTME-02A on the deck)               │
+  │         ├─ imu_link         (fixed, centre of base)                    │
+  │         ├─ ultrasonic_link  (fixed, HC-SR04 on the front)              │
+  │         ├─ door_left_link   / door_right_link   (revolute, grey doors) │
+  │         ├─ front_left_wheel_link / front_right_wheel_link (continuous)  │
+  │         └─ rear_left_wheel_link  / rear_right_wheel_link  (continuous)  │
   │                                                                         │
-  │  Ground clearance lowered (wheels closer to ground). Deck top 0.60 m.   │
+  │  Tiers: BLACK bottom box → GREY file compartment (split doors) →        │
+  │  BLACK top deck. Deck top 0.60 m; ground clearance lowered.             │
   └─────────────────────────────────────────────────────────────────────────┘
 -->
@@ -30,9 +29,8 @@
   <xacro:include filename="$(find my_robot_description)/urdf/wheels/drive_wheel.xacro"/>
   <xacro:include filename="$(find my_robot_description)/urdf/sensors/lidar.xacro"/>
-  <xacro:include filename="$(find my_robot_description)/urdf/sensors/rfid.xacro"/>
   <xacro:include filename="$(find my_robot_description)/urdf/sensors/imu.xacro"/>
   <xacro:include filename="$(find my_robot_description)/urdf/sensors/ultrasonic.xacro"/>
   <!-- ── Instantiate robot ── -->
-  <!-- Enclosure: base + compartment + split doors + frame + deck -->
+  <!-- Enclosure (base_link static geometry) + split doors -->
   <xacro:base/>
   <!-- 4WD skid-steer drive wheels (one per corner) -->
@@ -43,6 +41,5 @@
   <!-- Sensors -->
   <xacro:lidar/>        <!-- on the deck -->
-  <xacro:rfid/>         <!-- blue, deck edge -->
   <xacro:imu/>          <!-- centre of base -->
-  <xacro:ultrasonic/>   <!-- front "eyes" -->
+  <xacro:ultrasonic/>   <!-- HC-SR04 on the front -->
 </robot>
