Commit message: Phase 1 revision: black bottom box, grey split-door compartment (middle), black deck; RFID centred; HC-SR04 look; minimal TF (structural geometry merged onto base_link)
Co-Authored-By: Claude Opus 4.8 <noreply@anthropic.com>

File: src/my_robot_description/urdf/sensors/lidar.xacro (robot description, xacro)
@@ -2,8 +2,7 @@
 <!--
   LTME-02A lidar on the top deck. Frame "laser" (driver frame_id).
-  FIXED joint: the frame does not rotate in real use (driver outputs
-  de-rotated scans) so base->laser is on /tf_static — a continuous joint
-  would ride dynamic /tf at the joint-state rate and cause the 30 Hz scans
-  to be dropped by SLAM/Nav2.
+  FIXED joint (parented straight to base_link since the deck is not its own
+  frame): base->laser is on /tf_static — a moving joint would ride dynamic
+  /tf at the joint-state rate and the 30 Hz scans would be dropped by SLAM.
 -->
 <robot xmlns:xacro="http://www.ros.org/wiki/xacro">
@@ -21,9 +20,9 @@
       <xacro:cylinder_inertia_z m="${lidar_mass}" r="${lidar_radius}" h="${lidar_height}"/>
     </link>
-    <!-- Mounted on the deck top surface, centred (270° FOV faces forward). -->
+    <!-- On the deck top surface, centred (270° FOV faces forward). -->
     <joint name="laser_joint" type="fixed">
-      <parent link="deck_link"/>
+      <parent link="base_link"/>
       <child  link="laser"/>
-      <origin xyz="0 0 ${deck_thickness/2.0}" rpy="0 0 0"/>
+      <origin xyz="0 0 ${deck_top_z}" rpy="0 0 0"/>
     </joint>
   </xacro:macro>

File: src/my_robot_description/urdf/sensors/ultrasonic.xacro (robot description, xacro)
@@ -1,23 +1,36 @@
 <?xml version="1.0"?>
 <!--
-  HC-SR04 ultrasonic on the compartment front face, ~10 cm above ground,
-  pointing forward (+X). Modelled as the sensor's twin transducers — two
-  grey "eyes". Frame "ultrasonic_link" (frame_id of /ultrasonic/range) sits
-  at the pair centre with +X = measurement direction.
+  HC-SR04 ultrasonic on the front of the bottom box, ~10 cm above ground,
+  facing forward (+X). Modelled like the real module: a blue PCB, two black
+  cylindrical transducers ("eyes") protruding forward, and a silver crystal
+  can between them. Frame "ultrasonic_link" (frame_id of /ultrasonic/range)
+  sits on the board with +X = measurement direction.
 -->
 <robot xmlns:xacro="http://www.ros.org/wiki/xacro">
   <xacro:macro name="ultrasonic" params="">
     <link name="ultrasonic_link">
-      <!-- left eye -->
+      <!-- blue PCB -->
       <visual>
-        <origin xyz="0 ${us_eye_sep/2.0} 0" rpy="0 ${PI/2.0} 0"/>
-        <geometry><cylinder radius="${us_eye_radius}" length="${us_eye_length}"/></geometry>
-        <material name="ultrasonic_grey"/>
+        <origin xyz="0 0 0" rpy="0 0 0"/>
+        <geometry><box size="${us_pcb_t} ${us_pcb_w} ${us_pcb_h}"/></geometry>
+        <material name="us_pcb_blue"/>
       </visual>
-      <!-- right eye -->
+      <!-- left transducer (black cylinder, protruding forward) -->
       <visual>
-        <origin xyz="0 ${-us_eye_sep/2.0} 0" rpy="0 ${PI/2.0} 0"/>
-        <geometry><cylinder radius="${us_eye_radius}" length="${us_eye_length}"/></geometry>
-        <material name="ultrasonic_grey"/>
+        <origin xyz="${us_tx_length/2.0} ${us_tx_sep/2.0} 0" rpy="0 ${PI/2.0} 0"/>
+        <geometry><cylinder radius="${us_tx_radius}" length="${us_tx_length}"/></geometry>
+        <material name="us_transducer_black"/>
+      </visual>
+      <!-- right transducer -->
+      <visual>
+        <origin xyz="${us_tx_length/2.0} ${-us_tx_sep/2.0} 0" rpy="0 ${PI/2.0} 0"/>
+        <geometry><cylinder radius="${us_tx_radius}" length="${us_tx_length}"/></geometry>
+        <material name="us_transducer_black"/>
+      </visual>
+      <!-- silver crystal oscillator between the transducers -->
+      <visual>
+        <origin xyz="${us_pcb_t} 0 0" rpy="0 0 0"/>
+        <geometry><box size="0.005 0.010 0.005"/></geometry>
+        <material name="crystal_silver"/>
       </visual>
     </link>
@@ -25,5 +38,4 @@
       <parent link="base_link"/>
       <child  link="ultrasonic_link"/>
-      <!-- x: compartment front face; z: us_height_above_ground − wheel_radius -->
       <origin xyz="${body_length/2.0} 0 ${us_height_above_ground - wheel_radius}" rpy="0 0 0"/>
     </joint>

Commit message: Model revision 2: black full enclosure (bottom), grey corner bars, smaller raised grey file compartment with split doors, black deck; silver wheel hubs
Co-Authored-By: Claude Opus 4.8 <noreply@anthropic.com>

File: src/my_robot_description/urdf/base/base.xacro (robot description, xacro)
@@ -1,18 +1,17 @@
 <?xml version="1.0"?>
 <!--
-  Enclosure structure (chassis v3): a 3-tier file-delivery cabinet.
-  ALL static geometry is carried as multiple <visual> elements on base_link,
-  so it adds NO extra TF frames. Only the two doors (which move) get their own
-  links/frames.
-    tier 1  BLACK solid box     (bottom, no doors)
-    tier 2  GREY file compartment (hollow, open front) + split double-door
-    tier 3  BLACK deck board     (top surface; lidar + centred RFID sit on it)
+  Enclosure structure (chassis v3) — matches the real build.
+  All static geometry is carried as multiple <visual> elements on base_link,
+  so it adds NO extra TF frames. Only the two doors (which move) get frames.
+    tier 1  BLACK enclosure (full footprint, largest box)
+    (gap)   open — 4 GREY corner bars visible
+    tier 2  GREY file compartment (SMALLER, raised, hollow) + split double-door
+    tier 3  BLACK deck (full footprint, overhangs) — lidar + centred blue RFID
   TF frames from this file: base_footprint, base_link, door_left_link,
-  door_right_link.  (laser / imu_link / ultrasonic_link / wheels come from the
-  sensor & wheel macros.)
+  door_right_link.
 -->
 <robot xmlns:xacro="http://www.ros.org/wiki/xacro">
   <xacro:macro name="base" params="">
-    <!-- ── base_footprint (REP-105 ground projection) ── -->
+    <!-- ── base_footprint ── -->
     <link name="base_footprint"/>
     <joint name="base_joint" type="fixed">
@@ -27,33 +26,48 @@
         <geometry><box size="${body_length} ${body_width} ${chassis_thickness}"/></geometry>
         <material name="chassis_grey"/></visual>
-      <!-- tier 1: solid BLACK bottom box -->
-      <visual><origin xyz="0 0 ${bottom_black_center_z}"/>
-        <geometry><box size="${body_length} ${body_width} ${bottom_black_h}"/></geometry>
+      <!-- tier 1: BLACK bottom enclosure (full footprint, largest) -->
+      <visual><origin xyz="0 0 ${enclosure_center_z}"/>
+        <geometry><box size="${body_length} ${body_width} ${enclosure_h}"/></geometry>
         <material name="enclosure_black"/></visual>
-      <!-- tier 2: GREY file compartment — 5 panels, front open for the doors -->
-      <visual><origin xyz="0 0 ${compartment_center_z - compartment_h/2.0}"/>
-        <geometry><box size="${body_length} ${body_width} ${panel_thickness}"/></geometry>
-        <material name="compartment_grey"/></visual>                       <!-- floor -->
-      <visual><origin xyz="0 0 ${compartment_center_z + compartment_h/2.0}"/>
-        <geometry><box size="${body_length} ${body_width} ${panel_thickness}"/></geometry>
-        <material name="compartment_grey"/></visual>                       <!-- ceiling -->
-      <visual><origin xyz="${-body_length/2.0} 0 ${compartment_center_z}"/>
-        <geometry><box size="${panel_thickness} ${body_width} ${compartment_h}"/></geometry>
-        <material name="compartment_grey"/></visual>                       <!-- back -->
-      <visual><origin xyz="0 ${body_width/2.0} ${compartment_center_z}"/>
-        <geometry><box size="${body_length} ${panel_thickness} ${compartment_h}"/></geometry>
-        <material name="compartment_grey"/></visual>                       <!-- left -->
-      <visual><origin xyz="0 ${-body_width/2.0} ${compartment_center_z}"/>
-        <geometry><box size="${body_length} ${panel_thickness} ${compartment_h}"/></geometry>
-        <material name="compartment_grey"/></visual>                       <!-- right -->
-      <!-- tier 3: BLACK deck board (top surface) -->
+      <!-- 4 GREY corner bars (outer corners, full height enclosure→deck) -->
+      <xacro:property name="bx" value="${body_length/2.0 - bar_size/2.0}"/>
+      <xacro:property name="by" value="${body_width/2.0 - bar_size/2.0}"/>
+      <visual><origin xyz="${bx} ${by} ${bar_center_z}"/>
+        <geometry><box size="${bar_size} ${bar_size} ${bar_h}"/></geometry>
+        <material name="bar_grey"/></visual>
+      <visual><origin xyz="${bx} ${-by} ${bar_center_z}"/>
+        <geometry><box size="${bar_size} ${bar_size} ${bar_h}"/></geometry>
+        <material name="bar_grey"/></visual>
+      <visual><origin xyz="${-bx} ${by} ${bar_center_z}"/>
+        <geometry><box size="${bar_size} ${bar_size} ${bar_h}"/></geometry>
+        <material name="bar_grey"/></visual>
+      <visual><origin xyz="${-bx} ${-by} ${bar_center_z}"/>
+        <geometry><box size="${bar_size} ${bar_size} ${bar_h}"/></geometry>
+        <material name="bar_grey"/></visual>
+      <!-- tier 2: GREY file compartment (SMALLER) — 5 panels, front open -->
+      <visual><origin xyz="0 0 ${comp_bottom_z}"/>
+        <geometry><box size="${comp_length} ${comp_width} ${panel_thickness}"/></geometry>
+        <material name="compartment_grey"/></visual>                        <!-- floor -->
+      <visual><origin xyz="0 0 ${comp_top_z}"/>
+        <geometry><box size="${comp_length} ${comp_width} ${panel_thickness}"/></geometry>
+        <material name="compartment_grey"/></visual>                        <!-- ceiling -->
+      <visual><origin xyz="${-comp_length/2.0} 0 ${comp_center_z}"/>
+        <geometry><box size="${panel_thickness} ${comp_width} ${comp_h}"/></geometry>
+        <material name="compartment_grey"/></visual>                        <!-- back -->
+      <visual><origin xyz="0 ${comp_width/2.0} ${comp_center_z}"/>
+        <geometry><box size="${comp_length} ${panel_thickness} ${comp_h}"/></geometry>
+        <material name="compartment_grey"/></visual>                        <!-- left -->
+      <visual><origin xyz="0 ${-comp_width/2.0} ${comp_center_z}"/>
+        <geometry><box size="${comp_length} ${panel_thickness} ${comp_h}"/></geometry>
+        <material name="compartment_grey"/></visual>                        <!-- right -->
+      <!-- tier 3: BLACK deck board (full footprint, overhangs) -->
       <visual><origin xyz="0 0 ${deck_center_z}"/>
         <geometry><box size="${body_length} ${body_width} ${deck_h}"/></geometry>
         <material name="deck_black"/></visual>
-      <!-- RFID reader (blue), centred on the deck front-edge line -->
+      <!-- RFID reader (blue), centred on the deck -->
       <visual><origin xyz="${rfid_x} 0 ${deck_top_z + rfid_h/2.0}"/>
         <geometry><box size="${rfid_l} ${rfid_w} ${rfid_h}"/></geometry>
         <material name="rfid_blue"/></visual>
-      <collision><origin xyz="0 0 ${compartment_center_z}"/>
+      <collision><origin xyz="0 0 ${(struct_bottom_z + deck_top_z)/2.0}"/>
         <geometry><box size="${body_length} ${body_width} ${deck_top_z - struct_bottom_z}"/></geometry>
       </collision>
@@ -64,5 +78,5 @@
       <parent link="base_link"/>
       <child  link="door_left_link"/>
-      <origin xyz="${body_length/2.0} ${body_width/2.0} ${compartment_center_z}" rpy="0 0 0"/>
+      <origin xyz="${comp_length/2.0} ${comp_width/2.0} ${comp_center_z}" rpy="0 0 0"/>
       <axis xyz="0 0 1"/>
       <limit lower="0.0" upper="1.571" effort="2.0" velocity="2.0"/>
@@ -76,5 +90,5 @@
       <parent link="base_link"/>
       <child  link="door_right_link"/>
-      <origin xyz="${body_length/2.0} ${-body_width/2.0} ${compartment_center_z}" rpy="0 0 0"/>
+      <origin xyz="${comp_length/2.0} ${-comp_width/2.0} ${comp_center_z}" rpy="0 0 0"/>
       <axis xyz="0 0 1"/>
       <limit lower="-1.571" upper="0.0" effort="2.0" velocity="2.0"/>

File: src/my_robot_description/urdf/materials.xacro (robot description, xacro)
@@ -2,13 +2,8 @@
 <!-- Named materials for RViz visualisation (chassis v3 palette). -->
 <robot xmlns:xacro="http://www.ros.org/wiki/xacro">
-  <!-- Enclosure / bottom box / structure = black -->
+  <!-- Bottom enclosure + deck + lidar = black -->
   <material name="enclosure_black">
     <color rgba="0.08 0.08 0.09 1.0"/>
   </material>
-  <!-- File compartment (middle tier) + split doors = grey -->
-  <material name="compartment_grey">
-    <color rgba="0.55 0.55 0.57 1.0"/>
-  </material>
-  <!-- Top deck surface + lidar = black -->
   <material name="deck_black">
     <color rgba="0.10 0.10 0.11 1.0"/>
@@ -16,4 +11,12 @@
   <material name="lidar_black">
     <color rgba="0.06 0.06 0.07 1.0"/>
+  </material>
+  <!-- File compartment + split doors = grey -->
+  <material name="compartment_grey">
+    <color rgba="0.55 0.55 0.57 1.0"/>
+  </material>
+  <!-- Corner bars = grey (aluminium) -->
+  <material name="bar_grey">
+    <color rgba="0.72 0.73 0.75 1.0"/>
   </material>
   <!-- RFID reader = blue -->
@@ -31,10 +34,10 @@
     <color rgba="0.75 0.76 0.78 1.0"/>
   </material>
-  <!-- Wheels = black, hub accent -->
+  <!-- Wheels = black tyre, chrome/silver hub -->
   <material name="wheel_black">
     <color rgba="0.10 0.10 0.10 1.0"/>
   </material>
-  <material name="wheel_hub_blue">
-    <color rgba="0.20 0.20 0.80 1.0"/>
+  <material name="wheel_hub_silver">
+    <color rgba="0.80 0.82 0.85 1.0"/>
   </material>
   <!-- Chassis plate (hidden, low) -->

File: src/my_robot_description/urdf/properties.xacro (robot description, xacro)
@@ -4,19 +4,22 @@
   All distances in metres, masses in kg.  ROS REP-103: X fwd, Y left, Z up.
   base_link origin is at wheel-axis height above ground.
-  Enclosure (bottom → top):
-    tier 1  solid BLACK box (no doors)
-    tier 2  GREY file compartment (hollow) with a split double-door on the front
-    tier 3  BLACK top deck (surface) carrying the lidar + centred RFID reader
+  Enclosure layout (bottom → top), matching the real build:
+    tier 1  BLACK enclosure  — the largest box (full footprint)
+    (gap)   open, 4 GREY corner bars visible
+    tier 2  GREY file compartment — SMALLER footprint, raised & separated from
+            the enclosure, with a split double-door on the front
+    tier 3  BLACK top deck (overhangs) — carries lidar + centred blue RFID
+  The 4 grey bars run the full height (enclosure top → deck) at the outer
+  corners, so they are visible around the smaller compartment.
   Minimal TF: all static structure lives on base_link (multiple visuals) so it
-  produces NO extra TF frames. Only functional links get their own frame:
-  base_footprint, base_link, laser, imu_link, ultrasonic_link, the 4 wheels,
-  and the 2 (moving) doors.
+  produces NO extra frames. Only functional links get a frame: base_footprint,
+  base_link, laser, imu_link, ultrasonic_link, the 4 wheels, the 2 doors.
 -->
 <robot xmlns:xacro="http://www.ros.org/wiki/xacro">
   <!-- ── Math ── -->
   <xacro:property name="PI" value="3.14159265358979323846"/>
-  <!-- ── Footprint envelope ── -->
-  <xacro:property name="body_length"  value="0.400"/>   <!-- X 40 cm -->
-  <xacro:property name="body_width"   value="0.300"/>   <!-- Y 30 cm -->
+  <!-- ── Full footprint (bottom enclosure + top deck) ── -->
+  <xacro:property name="body_length"  value="0.400"/>   <!-- X -->
+  <xacro:property name="body_width"   value="0.300"/>   <!-- Y -->
   <xacro:property name="panel_thickness" value="0.012"/>
   <xacro:property name="chassis_thickness" value="0.020"/>
@@ -30,31 +33,40 @@
   <xacro:property name="ground_clearance" value="0.020"/>
   <xacro:property name="struct_bottom_z" value="${-(wheel_radius - ground_clearance)}"/> <!-- -0.045 -->
-  <!-- ── Tier heights (stack up from struct_bottom_z) ── -->
-  <xacro:property name="bottom_black_h" value="0.245"/>
-  <xacro:property name="compartment_h"  value="0.317"/>   <!-- grey file compartment -->
-  <xacro:property name="deck_h"         value="0.018"/>
-  <!-- Derived Z centres/levels (from base_link) -->
-  <xacro:property name="bottom_black_center_z" value="${struct_bottom_z + bottom_black_h/2.0}"/>          <!-- 0.0775 -->
-  <xacro:property name="bottom_black_top_z"    value="${struct_bottom_z + bottom_black_h}"/>              <!-- 0.200 -->
-  <xacro:property name="compartment_center_z"  value="${bottom_black_top_z + compartment_h/2.0}"/>        <!-- 0.3585 -->
-  <xacro:property name="compartment_top_z"     value="${bottom_black_top_z + compartment_h}"/>            <!-- 0.517 -->
-  <xacro:property name="deck_center_z"         value="${compartment_top_z + deck_h/2.0}"/>                <!-- 0.526 -->
-  <xacro:property name="deck_top_z"            value="${compartment_top_z + deck_h}"/>                    <!-- 0.535 → 0.600 ground -->
-  <!-- ── Split double-door (front of the GREY middle compartment) ── -->
-  <xacro:property name="door_height"    value="0.280"/>
-  <xacro:property name="door_width"     value="0.145"/>   <!-- each panel (Y) -->
+  <!-- ── Tier 1: BLACK bottom enclosure (full footprint) ── -->
+  <xacro:property name="enclosure_h" value="0.245"/>
+  <xacro:property name="enclosure_center_z" value="${struct_bottom_z + enclosure_h/2.0}"/>  <!-- 0.0775 -->
+  <xacro:property name="enclosure_top_z"    value="${struct_bottom_z + enclosure_h}"/>       <!-- 0.200 -->
+  <!-- ── Tier 3: BLACK top deck (full footprint, overhangs) ── -->
+  <xacro:property name="deck_h"        value="0.018"/>
+  <xacro:property name="deck_top_z"    value="0.535"/>                        <!-- 0.600 from ground -->
+  <xacro:property name="deck_bottom_z" value="${deck_top_z - deck_h}"/>       <!-- 0.517 -->
+  <xacro:property name="deck_center_z" value="${deck_top_z - deck_h/2.0}"/>   <!-- 0.526 -->
+  <!-- ── Grey corner bars (full height, outer corners) ── -->
+  <xacro:property name="bar_size"     value="0.020"/>
+  <xacro:property name="bar_h"        value="${deck_bottom_z - enclosure_top_z}"/>            <!-- 0.317 -->
+  <xacro:property name="bar_center_z" value="${(enclosure_top_z + deck_bottom_z)/2.0}"/>      <!-- 0.3585 -->
+  <!-- ── Tier 2: GREY file compartment (SMALLER, raised, split doors) ── -->
+  <xacro:property name="comp_length" value="0.280"/>   <!-- < body_length -->
+  <xacro:property name="comp_width"  value="0.200"/>   <!-- < body_width -->
+  <xacro:property name="comp_h"      value="0.200"/>
+  <xacro:property name="comp_top_z"    value="${deck_bottom_z}"/>                 <!-- ceiling touches deck: 0.517 -->
+  <xacro:property name="comp_center_z" value="${comp_top_z - comp_h/2.0}"/>       <!-- 0.417 -->
+  <xacro:property name="comp_bottom_z" value="${comp_top_z - comp_h}"/>           <!-- 0.317; open gap below to 0.200 -->
+  <!-- ── Split double-door (front of the GREY compartment) ── -->
+  <xacro:property name="door_height"    value="0.160"/>
+  <xacro:property name="door_width"     value="0.098"/>   <!-- each panel (Y), ~comp_width/2 -->
   <xacro:property name="door_thickness" value="0.012"/>
-  <!-- ── RFID reader (MFRC522) — centred on the deck front-edge line ── -->
+  <!-- ── RFID reader (MFRC522) — centred on the deck ── -->
   <xacro:property name="rfid_l" value="0.060"/>
   <xacro:property name="rfid_w" value="0.040"/>
   <xacro:property name="rfid_h" value="0.008"/>
-  <xacro:property name="rfid_x" value="${body_length/2.0 - rfid_l/2.0 - 0.02}"/>  <!-- front-edge line -->
+  <xacro:property name="rfid_x" value="${body_length/2.0 - rfid_l/2.0 - 0.03}"/>
   <!-- ── HC-SR04 ultrasonic (blue PCB + 2 black transducers + silver crystal) ── -->
-  <xacro:property name="us_pcb_w"    value="0.045"/>   <!-- board Y -->
-  <xacro:property name="us_pcb_h"    value="0.020"/>   <!-- board Z -->
-  <xacro:property name="us_pcb_t"    value="0.0015"/>  <!-- board X (thin) -->
-  <xacro:property name="us_tx_radius" value="0.008"/>  <!-- transducer can -->
+  <xacro:property name="us_pcb_w"    value="0.045"/>
+  <xacro:property name="us_pcb_h"    value="0.020"/>
+  <xacro:property name="us_pcb_t"    value="0.0015"/>
+  <xacro:property name="us_tx_radius" value="0.008"/>
   <xacro:property name="us_tx_length" value="0.012"/>
-  <xacro:property name="us_tx_sep"    value="0.026"/>  <!-- centre-to-centre -->
+  <xacro:property name="us_tx_sep"    value="0.026"/>
   <xacro:property name="us_height_above_ground" value="0.100"/>
   <!-- ── LTME-02A lidar (70 mm Ø, 60 mm tall) ── -->

File: src/my_robot_description/urdf/wheels/drive_wheel.xacro (robot description, xacro)
@@ -31,5 +31,5 @@
           <cylinder radius="${wheel_radius * 0.55}" length="${wheel_width * 1.05}"/>
         </geometry>
-        <material name="wheel_hub_blue"/>
+        <material name="wheel_hub_silver"/>
       </visual>
       <collision>
